File: ZigbeeShild01.kicad_pcb (KiCad board)
At the start: 2 copper layers, 65 x 30.5 mm, 27 parts, among them J1 Conn_01x06_Male, J2 RPi_GPIO, J3 Power, SW1 BSL, SW2 RST, U1 LM2596S-5, U2 AMS1117-3.3, U3 RF-BM-2652P2

Commit message: Gerber Files for production added
Other:
- board text added: "RF-BM-2652P2"

Commit message: some small changes in PCB
Routing:
- added copper zone on B.Cu, net GND
- added copper zone on F.Cu, net GND
